File: schematics/Bat Mgt Sys.kicad_sch (KiCad schematic)
At the start: 55 parts, among them J1 USB_C_Receptacle_PowerOnly_6P, J2 USB_A, Q1 IRLML6402, Q2 IRLML6402, U1 TPD1E05U06DPY, U2 TPD1E05U06DPY, U3 TPS2592xx, U4 TLV76701DRVx, U5 MCP6561-OT, U6 MCP6561-OT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

Commit message: Update schematics, add custom footprints, 3D models, and gitignore
Parts:
- removed U7: 74AHC1G02, symbol 74xGxx:74AHC1G02
- added C10, C9: 22, Capacitor_SMD:CP_Elec_6.3x5.4, symbol Device:C_Polarized_US
- added J3, J4: Screw_Terminal_01x02, bmslibs:OST_OSTTC020162, symbol Connector:Screw_Terminal_01x02
- added U8: 74AHC1G02W5-7, bmslibs:SOT95P280X140-5N, symbol 74AHC1G02W5-7:74AHC1G02W5-7
- HS1: footprint (none) -> bmslibs:SOT95P280X140-5N
- Thermistor(NXRT15XV103FA3A016)1: footprint (none) -> bmslibs:THROUGH_HOLES
Connections:
- net +BOUT: now also C9.1, J4.1 (Pin_1)
- net +POUT: now also C10.1, J3.1 (Pin_1), U8.5 (VCC)
- net GND: now also C10.2, C9.2, J3.2 (Pin_2), J4.2 (Pin_2), U8.3 (GND)
- net TH_OUT: now also U8.2 (B)
- net US_OUT: now also U8.1 (A)
- net VIN: now also U8.4 (Y)
Other:
- note added: "TH +"
- note added: "TH -"
