File: sim-lm311/sim-lm311.kicad_sch (KiCad schematic)
At the start: 17 parts, among them U1 74AHC1G02, U2 LM311D, U3 LM311D

Commit message: added ldo diagram
Connections:
- net LDO_IN: now reaches U1.4
Other:
- added sheet LDO part (untitled.kicad_sch)
Changed lines of the file:
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@@
+	(wire
+		(pts
+			(xy 128.27 143.51) (xy 134.62 143.51)
+		)
+		(stroke
+			(width 0)
+			(type default)
+		)
+	)
 	(wire
 		(pts
@@
 				)
 				(justify right)
+			)
+		)
+	)
+	(global_label "LDO_IN"
+		(shape input)
+		(at 134.62 143.51 0)
+		(fields_autoplaced yes)
+		(effects
+			(font
+				(size 1.27 1.27)
+			)
+			(justify left)
+		)
+		(property "Intersheetrefs" "${INTERSHEET_REFS}"
+			(at 144.1367 143.51 0)
+			(hide yes)
+			(show_name no)
+			(do_not_autoplace no)
+			(effects
+				(font
+					(size 1.27 1.27)
+				)
+				(justify left)
 			)
 		)
@@
 				)
 			)
+		)
+	)
+	(sheet
+		(at 238.76 152.4)
+		(size 15.24 3.81)
+		(exclude_from_sim no)
+		(in_bom yes)
+		(on_board yes)
+		(dnp no)
+		(fields_autoplaced yes)
+		(stroke
+			(width 0.1524)
+			(type solid)
+		)
+		(fill
+			(color 0 0 0 0)
+		)
+		(property "Sheetname" "LDO part"
+			(at 238.76 151.6884 0)
+			(show_name no)
+			(do_not_autoplace no)
+			(effects
+				(font
+					(size 1.27 1.27)
+				)
+				(justify left bottom)
+			)
+		)
+		(property "Sheetfile" "untitled.kicad_sch"
+			(at 238.76 156.7946 0)
+			(show_name no)
+			(do_not_autoplace no)
+			(effects
+				(font
+					(size 1.27 1.27)
+				)
+				(justify left top)
+			)
+		)
+		(instances
+			(project "sim-lm311"
+				(path "/9afa5773-09d4-4600-854f-3bd11830c8cf"
+					(page "2")
+				)
+			)
